File: KiCAD/K68-VDG.kicad_sch (KiCad schematic)
At the start: 48 parts

Commit message: 基板シルク印刷間違い訂正、回路図C1間違い訂正、v1.2ガーバー出力
Parts:
- C1, C10, C11, C12, C13, C4, C5, C6, C7, C8, C9: value (none) -> 0.1u; footprint (none) -> Capacitor_THT:C_Disc_D3.0mm_W1.6mm_P2.50mm
- C2: value (none) -> 10pF; footprint (none) -> Capacitor_THT:C_Disc_D3.0mm_W1.6mm_P2.50mm
- C3: value (none) -> 50pF; footprint (none) -> Capacitor_THT:C_Disc_D3.0mm_W1.6mm_P2.50mm
- D1: value (none) -> A13_LED; footprint (none) -> LED_THT:LED_D3.0mm
- D2: value (none) -> A14_LED; footprint (none) -> LED_THT:LED_D3.0mm
- D3: value (none) -> 1N4007; footprint (none) -> Diode_THT:D_DO-34_SOD68_P10.16mm_Horizontal
- H1, H2, H3, H4: value (none) -> MountingHole; footprint (none) -> MountingHole:MountingHole_3.2mm_M3
- J1: value (none) -> Video Out; footprint (none) -> RCA:RCAConAE
- J2: value (none) -> SBC6303 BUS; footprint (none) -> Connector_PinHeader_2.54mm:PinHeader_2x20_P2.54mm_Horizontal
- JP1: value (none) -> VRAM-JP; footprint (none) -> Jumper:SolderJumper-3_P1.3mm_Bridged12_RoundedPad1.0x1.5mm
- JP2: value (none) -> 8000-JP; footprint (none) -> Jumper:SolderJumper-2_P1.3mm_Open_RoundedPad1.0x1.5mm
- JP3: value (none) -> A000-JP; footprint (none) -> Jumper:SolderJumper-2_P1.3mm_Open_RoundedPad1.0x1.5mm
- Q1: value (none) -> 2SA1015; footprint (none) -> Package_TO_SOT_THT:TO-92_Inline_Wide
- Q2: value (none) -> 2SC1815; footprint (none) -> Package_TO_SOT_THT:TO-92_Inline_Wide
- R1: value (none) -> 1k; footprint (none) -> Resistor_THT:R_Axial_DIN0207_L6.3mm_D2.5mm_P5.08mm_Vertical
- R2: value (none) -> 360; footprint (none) -> Resistor_THT:R_Axial_DIN0207_L6.3mm_D2.5mm_P10.16mm_Horizontal
- R3: value (none) -> 560; footprint (none) -> Resistor_THT:R_Axial_DIN0207_L6.3mm_D2.5mm_P10.16mm_Horizontal
- R4: value (none) -> 3.9k; footprint (none) -> Resistor_THT:R_Axial_DIN0207_L6.3mm_D2.5mm_P10.16mm_Horizontal
- R5: value (none) -> 75; footprint (none) -> Resistor_THT:R_Axial_DIN0207_L6.3mm_D2.5mm_P10.16mm_Horizontal
- R6: value (none) -> 3.3k; footprint (none) -> Resistor_THT:R_Axial_DIN0207_L6.3mm_D2.5mm_P10.16mm_Horizontal
- R7: value (none) -> 470; footprint (none) -> Resistor_THT:R_Axial_DIN0207_L6.3mm_D2.5mm_P10.16mm_Horizontal
- R8, R9: value (none) -> 1k; footprint (none) -> Resistor_THT:R_Axial_DIN0207_L6.3mm_D2.5mm_P10.16mm_Horizontal
- RV1: value (none) -> 1k; footprint (none) -> Potentiometer_THT:Potentiometer_Vishay_T73YP_Vertical
- U1: value (none) -> MC6847; footprint (none) -> Package_DIP:DIP-40_W15.24mm_Socket_LongPads
- U10: value (none) -> 74LS138; footprint (none) -> Package_DIP:DIP-16_W7.62mm_Socket_LongPads
- U2: value (none) -> MC1372; footprint (none) -> Package_DIP:DIP-14_W7.62mm_Socket_LongPads
- U3: value (none) -> 74LS32; footprint (none) -> Package_DIP:DIP-14_W7.62mm_Socket_LongPads
- U4: value (none) -> 74HCT573; footprint (none) -> Package_DIP:DIP-20_W7.62mm_Socket_LongPads
- U5: value (none) -> 74LS02; footprint (none) -> Package_DIP:DIP-14_W7.62mm_Socket_LongPads
- U6, U9: value (none) -> 74LS244; footprint (none) -> Package_DIP:DIP-20_W7.62mm_Socket_LongPads
- U7: value (none) -> 74LS245; footprint (none) -> Package_DIP:DIP-20_W7.62mm_Socket_LongPads
- U8: value (none) -> 62256; footprint (none) -> Package_DIP:DIP-28_W15.24mm_Socket_LongPads
- Y1: value (none) -> 3.579545MHz; footprint (none) -> Crystal:Crystal_HC49-U_Vertical
Connections:
- net GND: now also C1.1
- net VCC: now also C1.2
Other:
- moved on the sheet: C1
